File: elec/layout/default/ams1117-33.kicad_pcb (KiCad board)
At the start: 2 copper layers, 225.7 x 100.8 mm, 0 parts

Commit message: initial design:
Parts:
- added C1: Multilayer Ceramic Capacitors MLCC - SMD/SMT 10uF 10V 0805 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, lib:C0805, F.Cu at (132.2, 74.5)
- added C2: Multilayer Ceramic Capacitors MLCC - SMD/SMT 10uF 10V 0805 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, lib:C0805, F.Cu at (132.0, 83.4)
- added U1: , lib:SOT-223-3_L6.5-W3.4-P2.30-LS7.0-BR, F.Cu at (132.2, 79.0)
Routing:
- net gnd: track 0.00 -> 16.4 mm
- net vcc-1: track 0.00 -> 11.7 mm
- net vcc: track 0.00 -> 3.86 mm
Changed lines of the file:
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@@
   )
   (net 0 "")
+  (net 1 "gnd")
+  (net 2 "vcc-1")
+  (net 3 "vcc")
+  (footprint "lib:SOT-223-3_L6.5-W3.4-P2.30-LS7.0-BR" (layer "F.Cu")
+    (at 132.175 78.95)
+    (attr smd)
+    (fp_text reference "U1" (at -2.683474 -2.834775) (layer "F.SilkS")
+        (effects (font (size 1 1) (thickness 0.15)))
+    )
+    (fp_text value "" (at 0 6.3) (layer "F.Fab")
+        (effects (font (size 1 1) (thickness 0.15)))
+    )
+    (fp_text user "${REFERENCE}" (at 0 0) (layer "F.Fab")
+        (effects (font (size 1 1) (thickness 0.15)))
+    )
+    (fp_line (start -1.57 -3.33) (end 1.37 -3.33)
+      (stroke (width 0.15) (type solid)) (layer "F.SilkS"))
+    (fp_line (start -1.57 3.33) (end -1.57 -3.33)
+      (stroke (width 0.15) (type solid)) (layer "F.SilkS"))
+    (fp_line (start 1.37 -3.33) (end 1.37 3.33)
+      (stroke (width 0.15) (type solid)) (layer "F.SilkS"))
+    (fp_line (start 1.37 3.33) (end -1.57 3.33)
+      (stroke (width 0.15) (type solid)) (layer "F.SilkS"))
+    (fp_circle (center 4.55 2.19) (end 4.8 2.19)
+      (stroke (width 0.5) (type solid)) (fill none) (layer "Cmts.User"))
+    (fp_circle (center 3.4 3.25) (end 3.43 3.25)
+      (stroke (width 0.06) (type solid)) (fill none) (layer "F.Fab"))
+    (pad "1" smd rect (at 2.97 2.3) (size 2.5 1.1) (layers "F.Cu" "F.Paste" "F.Mask")
+      (net 1 "gnd") (pintype "stereo"))
+    (pad "2" smd rect (at 2.97 0) (size 2.5 1.1) (layers "F.Cu" "F.Paste" "F.Mask")
+      (net 2 "vcc-1") (pintype "stereo"))
+    (pad "3" smd rect (at 2.97 -2.3) (size 2.5 1.1) (layers "F.Cu" "F.Paste" "F.Mask")
+      (net 3 "vcc") (pintype "stereo"))
+    (pad "4" smd rect (at -2.97 0) (size 2.34 3.6) (layers "F.Cu" "F.Paste" "F.Mask")
+      (net 2 "vcc-1") (pintype "stereo"))
+    (model "/Users/narayanpowderly/Documents/atopile-workspace/swoop/.ato/modules/ams1117-33/elec/footprints/footprints.3dshapes/SOT-223-4P_L6.5-W3.5-H1.6-LS7.0-P2.30.wrl"
+      (offset (xyz -3.99 2.92 -0))
+      (scale (xyz 1 1 1))
+      (rotate (xyz 0 0 180))
+    )
+  )
+  (footprint "lib:C0805" (layer "F.Cu")
+    (at 132.000375 83.433928)
+    (descr "Capacitor SMD 0805 (2012 Metric), square (rectangular) end terminal, IPC_7351 nominal, (Body size source: IPC-SM-782 page 76, https://www.pcb-3d.com/wordpress/wp-content/uploads/ipc-sm-782a_amendment_1_and_2.pdf, https://docs.google.com/spreadsheets/d/1BsfQQcO9C6DZCsRaXUlFlo91Tg2WpOkGARC1WS5S8t0/edit?usp=sharing), generated with kicad-footprint-generator")
+    (tags "capacitor")
+    (attr smd)
+    (fp_text reference "C2" (at 2.872171 0.026229) (layer "F.SilkS")
+        (effects (font (size 1 1) (thickness 0.15)))
+    )
+    (fp_text value "Multilayer Ceramic Capacitors MLCC - SMD/SMT 10uF 10V 0805 RoHS" (at 0 1.68) (layer "F.Fab")
+        (effects (font (size 1 1) (thickness 0.15)))
+    )
+    (fp_text user "${REFERENCE}" (at 0 0) (layer "F.Fab")
+        (effects (font (size 0.5 0.5) (thickness 0.08)))
+    )
+    (fp_line (start -0.261252 -0.735) (end 0.261252 -0.735)
+      (stroke (width 0.12) (type solid)) (layer "F.SilkS"))
+    (fp_line (start -0.261252 0.735) (end 0.261252 0.735)
+      (stroke (width 0.12) (type solid)) (layer "F.SilkS"))
+    (fp_line (start -1.7 -0.98) (end 1.7 -0.98)
+      (stroke (width 0.05) (type solid)) (layer "F.CrtYd"))
+    (fp_line (start -1.7 0.98) (end -1.7 -0.98)
+      (stroke (width 0.05) (type solid)) (layer "F.CrtYd"))
+    (fp_line (start 1.7 -0.98) (end 1.7 0.98)
+      (stroke (width 0.05) (type solid)) (layer "F.CrtYd"))
+    (fp_line (start 1.7 0.98) (end -1.7 0.98)
+      (stroke (width 0.05) (type solid)) (layer "F.CrtYd"))
+    (fp_line (start -1 -0.625) (end 1 -0.625)
+      (stroke (width 0.1) (type solid)) (layer "F.Fab"))
+    (fp_line (start -1 0.625) (end -1 -0.625)
+      (stroke (width 0.1) (type solid)) (layer "F.Fab"))
+    (fp_line (start 1 -0.625) (end 1 0.625)
+      (stroke (width 0.1) (type solid)) (layer "F.Fab"))
+    (fp_line (start 1 0.625) (end -1 0.625)
+      (stroke (width 0.1) (type solid)) (layer "F.Fab"))
+    (pad "1" smd roundrect (at -0.95 0) (size 1 1.45) (layers "F.Cu" "F.Paste" "F.Mask") (roundrect_rratio 0.25)
+      (net 2 "vcc-1") (pintype "stereo"))
+    (pad "2" smd roundrect (at 0.95 0) (size 1 1.45) (layers "F.Cu" "F.Paste" "F.Mask") (roundrect_rratio 0.25)
+      (net 1 "gnd") (pintype "stereo"))
+    (model "${KICAD6_3DMODEL_DIR}/Capacitor_SMD.3dshapes/C_0805_2012Metric.wrl"
+      (offset (xyz 0 0 0))
+      (scale (xyz 1 1 1))
+      (rotate (xyz 0 0 0))
+    )
+  )
+  (footprint "lib:C0805" (layer "F.Cu")
+    (at 132.198399 74.461913 180)
+    (descr "Capacitor SMD 0805 (2012 Metric), square (rectangular) end terminal, IPC_7351 nominal, (Body size source: IPC-SM-782 page 76, https://www.pcb-3d.com/wordpress/wp-content/uploads/ipc-sm-782a_amendment_1_and_2.pdf, https://docs.google.com/spreadsheets/d/1BsfQQcO9C6DZCsRaXUlFlo91Tg2WpOkGARC1WS5S8t0/edit?usp=sharing), generated with kicad-footprint-generator")
+    (tags "capacitor")
+    (attr smd)
+    (fp_text reference "C1" (at -2.804591 -0.073359) (layer "F.SilkS")
+        (effects (font (size 1 1) (thickness 0.15)))
+    )
+    (fp_text value "Multilayer Ceramic Capacitors MLCC - SMD/SMT 10uF 10V 0805 RoHS" (at 0 1.68) (layer "F.Fab")
+        (effects (font (size 1 1) (thickness 0.15)))
+    )
+    (fp_text user "${REFERENCE}" (at 0 0) (layer "F.Fab")
+        (effects (font (size 0.5 0.5) (thickness 0.08)))
+    )
+    (fp_line (start -0.261252 -0.735) (end 0.261252 -0.735)
+      (stroke (width 0.12) (type solid)) (layer "F.SilkS"))
+    (fp_line (start -0.261252 0.735) (end 0.261252 0.735)
+      (stroke (width 0.12) (type solid)) (layer "F.SilkS"))
+    (fp_line (start -1.7 -0.98) (end 1.7 -0.98)
+      (stroke (width 0.05) (type solid)) (layer "F.CrtYd"))
+    (fp_line (start -1.7 0.98) (end -1.7 -0.98)
+      (stroke (width 0.05) (type solid)) (layer "F.CrtYd"))
+    (fp_line (start 1.7 -0.98) (end 1.7 0.98)
+      (stroke (width 0.05) (type solid)) (layer "F.CrtYd"))
+    (fp_line (start 1.7 0.98) (end -1.7 0.98)
+      (stroke (width 0.05) (type solid)) (layer "F.CrtYd"))
+    (fp_line (start -1 -0.625) (end 1 -0.625)
+      (stroke (width 0.1) (type solid)) (layer "F.Fab"))
+    (fp_line (start -1 0.625) (end -1 -0.625)
+      (stroke (width 0.1) (type solid)) (layer "F.Fab"))
+    (fp_line (start 1 -0.625) (end 1 0.625)
+      (stroke (width 0.1) (type solid)) (layer "F.Fab"))
+    (fp_line (start 1 0.625) (end -1 0.625)
+      (stroke (width 0.1) (type solid)) (layer "F.Fab"))
+    (pad "1" smd roundrect (at -0.95 0 180) (size 1 1.45) (layers "F.Cu" "F.Paste" "F.Mask") (roundrect_rratio 0.25)
+      (net 3 "vcc") (pintype "stereo"))
+    (pad "2" smd roundrect (at 0.95 0 180) (size 1 1.45) (layers "F.Cu" "F.Paste" "F.Mask") (roundrect_rratio 0.25)
+      (net 1 "gnd") (pintype "stereo"))
+    (model "${KICAD6_3DMODEL_DIR}/Capacitor_SMD.3dshapes/C_0805_2012Metric.wrl"
+      (offset (xyz 0 0 0))
+      (scale (xyz 1 1 1))
+      (rotate (xyz 0 0 0))
+    )
+  )
   (gr_circle (center 225.62 81.79) (end 227.32 81.79)
     (stroke (width 0.1) (type solid)) (fill none) (layer "Edge.Cuts"))
@@
       (xy 69.100734 49.778315)
     )
-    (stroke (width 0) (type solid)) (fill none) (layer "Edge.Cuts"))
+    (stroke (width 0.1) (type solid)) (fill none) (layer "Edge.Cuts"))
   (gr_arc (start 261.62 113.79) (mid 260.448427 116.618427) (end 257.62 117.79)
     (stroke (width 0.1) (type solid)) (layer "Edge.Cuts"))
@@
     (effects (font (size 2 2) (thickness 0.1)) (justify left bottom))
   )
+  (segment (start 133.918118 83.433928) (end 132.950375 83.433928) (width 1) (layer "F.Cu") (net 1))
+  (segment (start 135.145 81.25) (end 135.134303 81.25) (width 0.25) (layer "F.Cu") (net 1))
+  (segment (start 135.134303 82.217743) (end 133.918118 83.433928) (width 1) (layer "F.Cu") (net 1))
+  (segment (start 131.248399 75.798399) (end 133.19155 77.74155) (width 0.5) (layer "F.Cu") (net 1))
+  (segment (start 136.296395 81.25) (end 135.145 81.25) (width 0.5) (layer "F.Cu") (net 1))
+  (segment (start 137.035375 80.51102) (end 136.296395 81.25) (width 0.5) (layer "F.Cu") (net 1))
+  (segment (start 131.248399 74.461913) (end 131.248399 75.798399) (width 0.5) (layer "F.Cu") (net 1))
+  (segment (start 137.035375 78.08166) (end 137.035375 80.51102) (width 0.5) (layer "F.Cu") (net 1))
+  (segment (start 136.695265 77.74155) (end 137.035375 78.08166) (width 0.5) (layer "F.Cu") (net 1))
+  (segment (start 135.134303 81.25) (end 135.134303 82.217743) (width 1) (layer "F.Cu") (net 1))
+  (segment (start 133.19155 77.74155) (end 136.695265 77.74155) (width 0.5) (layer "F.Cu") (net 1))
+  (segment (start 130.102151 83.433928) (end 129.205 82.536777) (width 1) (layer "F.Cu") (net 2))
+  (segment (start 129.205 82.536777) (end 129.205 78.95) (width 1) (layer "F.Cu") (net 2))
+  (segment (start 135.145 78.95) (end 129.205 78.95) (width 1) (layer "F.Cu") (net 2))
+  (segment (start 131.050375 83.433928) (end 130.102151 83.433928) (width 1) (layer "F.Cu") (net 2))
+  (segment (start 133.148399 74.461913) (end 133.148399 76.089584) (width 1) (layer "F.Cu") (net 3))
+  (segment (start 133.708815 76.65) (end 135.145 76.65) (width 1) (layer "F.Cu") (net 3))
+  (segment (start 133.148399 76.089584) (end 133.708815 76.65) (width 1) (layer "F.Cu") (net 3))
   (group "" (id 6c1ef9f7-0f34-47bb-ac1a-76df23fb396e)
     (members

Commit message: update layout
Parts:
- C1, C2: value Multilayer Ceramic Capacitors MLCC - SMD/SMT 10uF 10V 0805 RoHS -> 25V 10uF X5R ±10% 0805 Multilayer Ceramic Capacitors MLCC - SMD/SMT ROHS
Changed lines of the file:
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@@
         (effects (font (size 1 1) (thickness 0.15)))
     )
-    (fp_text value "Multilayer Ceramic Capacitors MLCC - SMD/SMT 10uF 10V 0805 RoHS" (at 0 1.68) (layer "F.Fab")
+    (fp_text value "25V 10uF X5R ±10% 0805  Multilayer Ceramic Capacitors MLCC - SMD/SMT ROHS" (at 0 1.68) (layer "F.Fab")
         (effects (font (size 1 1) (thickness 0.15)))
     )
@@
         (effects (font (size 1 1) (thickness 0.15)))
     )
-    (fp_text value "Multilayer Ceramic Capacitors MLCC - SMD/SMT 10uF 10V 0805 RoHS" (at 0 1.68) (layer "F.Fab")
+    (fp_text value "25V 10uF X5R ±10% 0805  Multilayer Ceramic Capacitors MLCC - SMD/SMT ROHS" (at 0 1.68) (layer "F.Fab")
         (effects (font (size 1 1) (thickness 0.15)))
     )
